Commit message: Tested with gazebo fortress

File: src/bot_description/urdf/bot.urdf.xacro (robot description, xacro)
@@ -2,4 +2,8 @@
 <robot xmlns:xacro="http://www.ros.org/wiki/xacro" name="ylvov_robot">
     <xacro:include filename="$(find bot_description)/urdf/properties.xacro" />
-	<xacro:include filename="$(find bot_description)/urdf/base.xacro" />
+	<xacro:include filename="$(find bot_description)/urdf/materials.xacro" />
+	<xacro:include filename="$(find bot_description)/urdf/macros.xacro" />
+	<xacro:include filename="$(find bot_description)/urdf/links.xacro" />
+	<xacro:include filename="$(find bot_description)/urdf/joints.xacro" />
+	<!-- <xacro:include filename="$(find bot_description)/urdf/bot.gazebo.xacro" /> -->
 </robot>

File: src/bot_description/urdf/properties.xacro (robot description, xacro)
@@ -1,6 +1,15 @@
 <?xml version="1.0"?>
 <robot xmlns:xacro="http://www.ros.org/wiki/xacro">
-    <xacro:property name="base_length" value="0.5" />
-    <xacro:property name="base_width" value="0.5" />
-    <xacro:property name="base_height" value="0.5" />
+    <xacro:property name="base_length" value="0.2" />
+    <xacro:property name="base_width" value="0.15" />
+    <xacro:property name="base_height" value="0.03" />
+    <xacro:property name="base_mass" value="1" />
+    <xacro:property name="engine_length" value="0.06" />
+    <xacro:property name="engine_width" value="0.03" />
+    <xacro:property name="engine_height" value="0.03" />
+    <xacro:property name="engine_mass" value="0.1" />
+    <xacro:property name="shaft_length" value="0.004" />
+    <xacro:property name="shaft_radius" value="0.003" />
+    <xacro:property name="wheel_length" value="0.02" />
+    <xacro:property name="wheel_radius" value="0.035" />
 </robot>
